Commit message: Origin of PointCloud is actually "camera_color_optical_frame", have to shift "camera_link".

File: robot_model/mpo_700/xacros/depth_camera.xacro (robot description, xacro)
@@ -22,5 +22,5 @@
 			    </collision>
 			    <visual>
-			      <origin xyz="0 -0.0175 0" rpy="1.570796 0 1.570796"/>
+			      <origin xyz="0 -0.0325 0" rpy="1.570796 0 1.570796"/>
 			      <geometry>
 			      	<mesh filename="package://neo_mpo_700/robot_model/mpo_700/meshes/d435.dae"/>

Commit message: New link added for fixing issues in simulation.

File: robot_model/mpo_700/xacros/depth_camera.xacro (robot description, xacro)
@@ -10,7 +10,12 @@
 		    </joint>
 		    <joint name="${name}_optical_joint" type="fixed">
-		    	<origin xyz="0 0 0" rpy="${-pi/2} 0 ${-pi/2}"/>
+		    	<origin xyz="0 0.015 0" rpy="${-pi/2} 0 ${-pi/2}"/>
 		    	<parent link="${name}_link"/>
 		    	<child link="${name}_link_optical"/>
+		    </joint>
+		    <joint name="${name}_gazebo_joint" type="fixed">
+		    	<origin xyz="0 0.015 0" rpy="0 0 0"/>
+		    	<parent link="${name}_link"/>
+		    	<child link="${name}_link_gazebo"/>
 		    </joint>
 		    <link name="${name}_link">
@@ -38,4 +43,5 @@
 		    <link  name="${name}_link_optical">
 		    </link>
+		    <link name="${name}_link_gazebo" />
 	</xacro:macro>
 </robot>

File: robot_model/mpo_700/xacros/mpo_700_gazebo.xacro (robot description, xacro)
@@ -75,5 +75,5 @@
         </sensor>
   </gazebo>
-    <gazebo reference="imu_link">
+  <gazebo reference="imu_link">
     <gravity>true</gravity>
     <sensor name="imu_sensor" type="imu">
@@ -94,5 +94,15 @@
     </sensor>
   </gazebo>
-    <!-- camera -->
+ <gazebo>
+    <plugin name="mpo_700_controller" filename="libgazebo_ros_planar_move.so">
+      <commandTopic>cmd_vel</commandTopic>
+      <odometryTopic>odom</odometryTopic>
+      <odometryFrame>odom</odometryFrame>
+      <odometryRate>150.0</odometryRate>
+      <robotBaseFrame>base_link</robotBaseFrame>
+    </plugin>
+  </gazebo>
+  <!-- camera -->
+  <!-->
   <gazebo reference="camera_link">
     <sensor type="camera" name="camera1">
@@ -100,7 +110,47 @@
       <camera name="head">
         <horizontal_fov>1.3962634</horizontal_fov>
+  <image>
+    <width>800</width>
+    <height>800</height>
+    <format>R8G8B8</format>
+  </image>
+        <clip>
+          <near>0.02</near>
+          <far>300</far>
+        </clip>
+        <noise>
+          <type>gaussian</type>
+           Noise is sampled independently per pixel on each frame.
+               That pixel's noise value is added to each of its color
+               channels, which at that point lie in the range [0,1].
+          <mean>0.0</mean>
+          <stddev>0.007</stddev>
+        </noise>
+      </camera>
+      <plugin name="camera_controller" filename="libgazebo_ros_camera.so">
+        <alwaysOn>true</alwaysOn>
+        <updateRate>0.0</updateRate>
+        <cameraName>robot/camera1</cameraName>
+        <imageTopicName>image_raw</imageTopicName>
+        <cameraInfoTopicName>camera_info</cameraInfoTopicName>
+        <frameName>camera_link</frameName>
+        <hackBaseline>0.07</hackBaseline>
+        <distortionK1>0.0</distortionK1>
+        <distortionK2>0.0</distortionK2>
+        <distortionK3>0.0</distortionK3>
+        <distortionT1>0.0</distortionT1>
+        <distortionT2>0.0</distortionT2>
+      </plugin>
+    </sensor>
+  </gazebo>
+  <-->
+  <gazebo reference="camera_link_gazebo">
+    <sensor name="camera1" type="depth">
+      <update_rate>15</update_rate>
+      <hfov>70</hfov>
+      <camera name="head">
         <image>
-          <width>800</width>
-          <height>800</height>
+          <width>320</width>
+          <height>240</height>
           <format>R8G8B8</format>
         </image>
@@ -115,31 +165,68 @@
                channels, which at that point lie in the range [0,1]. -->
           <mean>0.0</mean>
-          <stddev>0.007</stddev>
+          <stddev>0.03</stddev>
         </noise>
       </camera>
-      <plugin name="camera_controller" filename="libgazebo_ros_camera.so">
+      <plugin name="camera1_controller" filename="libgazebo_ros_openni_kinect.so">
+        <!--<baseline>0.2</baseline>-->
         <alwaysOn>true</alwaysOn>
         <updateRate>0.0</updateRate>
-        <cameraName>camera1</cameraName>
-        <imageTopicName>image_raw</imageTopicName>
-        <cameraInfoTopicName>camera_info</cameraInfoTopicName>
-        <frameName>camera_link</frameName>
-        <hackBaseline>0.07</hackBaseline>
-        <distortionK1>0.0</distortionK1>
-        <distortionK2>0.0</distortionK2>
-        <distortionK3>0.0</distortionK3>
-        <distortionT1>0.0</distortionT1>
-        <distortionT2>0.0</distortionT2>
+        <cameraName>camera_ir</cameraName>
+        <imageTopicName>/camera/depth/image_raw</imageTopicName>
+        <cameraInfoTopicName>/camera/depth/camera_info</cameraInfoTopicName>
+        <depthImageTopicName>/camera/depth/depth_raw</depthImageTopicName>
+        <depthImageInfoTopicName>/camera/depth/camera_info</depthImageInfoTopicName>
+        <pointCloudTopicName>/camera/depth_registered/points</pointCloudTopicName>
+        <frameName>camera_link_optical</frameName>
+        <pointCloudCutoff>0.12</pointCloudCutoff>
+        <pointCloudCutoffMax>3.0</pointCloudCutoffMax>
+        <distortionK1>0.00000001</distortionK1>
+        <distortionK2>0.00000001</distortionK2>
+        <distortionK3>0.00000001</distortionK3>
+        <distortionT1>0.00000001</distortionT1>
+        <distortionT2>0.00000001</distortionT2>
+        <CxPrime>0</CxPrime>
+        <Cx>0</Cx>
+        <Cy>0</Cy>
+        <focalLength>0</focalLength>
+        <hackBaseline>0</hackBaseline>
       </plugin>
     </sensor>
   </gazebo>
- <gazebo>
-    <plugin name="mpo_700_controller" filename="libgazebo_ros_planar_move.so">
-      <commandTopic>cmd_vel</commandTopic>
-      <odometryTopic>odom</odometryTopic>
-      <odometryFrame>odom</odometryFrame>
-      <odometryRate>20.0</odometryRate>
-      <robotBaseFrame>base_link</robotBaseFrame>
-    </plugin>
+  <!-- Sonar -->
+  <gazebo reference="us_1_link">
+  <!-- Visuals / Collisions omitted for this example -->
+  <sensor type="ray" name="range">
+    <ray>
+         <scan>
+            <horizontal>
+               <samples>1</samples>
+               <resolution>1.0</resolution>
+               <min_angle>-0.01</min_angle>
+               <max_angle>0.01</max_angle>
+            </horizontal>
+            <vertical>
+               <samples>1</samples>
+               <resolution>1</resolution>
+               <min_angle>-0.01</min_angle>
+               <max_angle>0.01</max_angle>
+            </vertical>
+         </scan>
+         <range>
+            <min>0.01</min>
+            <max>3.75</max>
+            <resolution>0.02</resolution>
+         </range>
+      </ray>
+      <plugin filename="libgazebo_ros_range.so" name="gazebo_ros_range">
+  <gaussianNoise>0.005</gaussianNoise>
+  <alwaysOn>true</alwaysOn>
+  <updateRate>50</updateRate>
+  <topicName>ultrasonic/us1</topicName>
+  <frameName>us_1_link</frameName>
+  <radiation>INFRARED</radiation>
+  <fov>0.2967</fov>
+      </plugin>
+      </sensor>
   </gazebo>
 </robot>
