Commit message: The model now should fit the real camera model.

File: robot_model/mpo_700/mpo_700.urdf.xacro (robot description, xacro)
@@ -128,5 +128,5 @@
   <!-- Depth Camera -->
   <!-- xacro:depth_camera name="camera" parent="base_link">
-    <origin xyz="0.228 0 0.461" rpy="0 0 0" />
+    <origin xyz="0.228 -0.015 0.461" rpy="0 0 0" />
   </xacro:depth_camera-->
 </robot>

File: robot_model/mpo_700/xacros/depth_camera.xacro (robot description, xacro)
@@ -22,5 +22,5 @@
 			    </collision>
 			    <visual>
-			      <origin xyz="0 -0.0325 0" rpy="1.570796 0 1.570796"/>
+			      <origin xyz="0 -0.0175 0" rpy="1.570796 0 1.570796"/>
 			      <geometry>
 			      	<mesh filename="package://neo_mpo_700/robot_model/mpo_700/meshes/d435.dae"/>

Commit message: New monting setup of camera.

File: robot_model/mpo_700/mpo_700.urdf.xacro (robot description, xacro)
@@ -128,5 +128,5 @@
   <!-- Depth Camera -->
   <!-- xacro:depth_camera name="camera" parent="base_link">
-    <origin xyz="0.228 -0.015 0.461" rpy="0 0 0" />
+    <origin xyz="-0.228 0.015 0.461" rpy="0 0 3.14159" />
   </xacro:depth_camera-->
 </robot>
